Commit message: Update bringup pkg

File: fourbox_description/description/properties.xacro (robot description, xacro)
@@ -7,9 +7,8 @@
     <xacro:property name="wheel_mass" value="0.1" />
     <xacro:property name="wheel_count" value="4" />
-    <xacro:property name="wheel_radius" value="0.0325" />
+    <xacro:property name="wheel_radius" value="0.033" />
     <xacro:property name="wheel_length" value="0.025" />
-    <xacro:property name="wheel_separation_x" value="0.21" />
-    <xacro:property name="wheel_separation_y" value="0.166" />
-    <!-- <xacro:property name="correction_coefficient_with_wheel" value="0.01" /> -->
+    <xacro:property name="wheel_separation_x" value="0.210" />
+    <xacro:property name="wheel_separation_y" value="0.165" />
     <xacro:property name="lidar_mass" value="0.1" />
     <xacro:property name="lidar_length" value="0.025" />

File: fourbox_description/description/ros2_control.xacro (robot description, xacro)
@@ -8,8 +8,8 @@
         <param name="baudrate">$(arg baudrate_arg)</param>
         <param name="serial_port_name">$(arg serial_port_name_arg)</param>
-        <param name="wheel_count">"${wheel_count}"</param>
-        <param name="wheel_radius">"${wheel_radius}"</param>
-        <param name="wheel_separation_x">"${wheel_separation_x}"</param>
-        <param name="wheel_separation_y">"${wheel_separation_y}"</param>
+        <param name="wheel_count">${wheel_count}</param>
+        <param name="wheel_radius">${wheel_radius}</param>
+        <param name="wheel_separation_x">${wheel_separation_x}</param>
+        <param name="wheel_separation_y">${wheel_separation_y}</param>
         </hardware>
         <joint name="base_front_left_wheel_joint">
