Commit message: Update bringup pkg

File: fourbox_description/description/fourbox.urdf.xacro (robot description, xacro)
@@ -3,4 +3,7 @@
     <!-- Параметры -->
     <!-- <xacro:arg name="use_simulation" default="false" /> -->
+    <xacro:arg name="encoder_ppr_arg" default="988"/>
+    <xacro:arg name="baudrate_arg" default="115200"/>
+    <xacro:arg name="serial_port_name_arg" default="/dev/ttyUSB0"/>
     <!-- Вспомогательные модули -->
     <xacro:include filename="materials.xacro" />

File: fourbox_description/description/properties.xacro (robot description, xacro)
@@ -6,4 +6,5 @@
     <xacro:property name="base_height" value="0.11" />
     <xacro:property name="wheel_mass" value="0.1" />
+    <xacro:property name="wheel_count" value="4" />
     <xacro:property name="wheel_radius" value="0.0325" />
     <xacro:property name="wheel_length" value="0.025" />

File: fourbox_description/description/ros2_control.xacro (robot description, xacro)
@@ -1,17 +1,16 @@
 <?xml version="1.0"?>
 <robot xmlns:xacro="http://www.ros.org/wiki/xacro" name="lidar">
-    <!-- ✅ КРИТИЧЕСКИ ВАЖНО! ros2_control секция -->
     <ros2_control name="FourboxSystem" type="system">
         <hardware>
-        <plugin>fourbox_hardware/FourboxHardware</plugin>
-        <!-- ✅ Параметры hardware из config/robot_hardware.yaml -->
-        <param name="serial_port">/dev/ttyUSB0</param>
-        <param name="baudrate">115200</param>
-        <param name="wheel_radius">0.1</param>
-        <param name="wheel_separation_horizontal">0.4</param>
-        <param name="wheel_separation_vertical">0.5</param>
-        <param name="encoder_ppr">988</param>
+        <plugin>dasrobot_drive_controller/DasrobotDriveController</plugin>
+        <!-- <plugin>fourbox_hardware/FourboxHardware</plugin> -->
+        <param name="encoder_ppr">$(arg encoder_ppr_arg)</param>
+        <param name="baudrate">$(arg baudrate_arg)</param>
+        <param name="serial_port_name">$(arg serial_port_name_arg)</param>
+        <param name="wheel_count">"${wheel_count}"</param>
+        <param name="wheel_radius">"${wheel_radius}"</param>
+        <param name="wheel_separation_x">"${wheel_separation_x}"</param>
+        <param name="wheel_separation_y">"${wheel_separation_y}"</param>
         </hardware>
-        <!-- ✅ Интерфейсы для Mecanum контроллера -->
         <joint name="base_front_left_wheel_joint">
         <command_interface name="velocity"/>

Commit message: Added launch files

File: fourbox_description/description/fourbox.urdf.xacro (robot description, xacro)
@@ -15,5 +15,5 @@
     <xacro:include filename="lidar.xacro" />
     <!-- Подключаемые модули -->
-    <xacro:include filename="ros2_control.xacro" />
+    <!-- <xacro:include filename="ros2_control.xacro" /> -->
     <!-- <xacro:if value="$(arg use_simulation)">
         <xacro:include filename="gazebo_plugins.xacro" />

File: fourbox_description/description/lidar.xacro (robot description, xacro)
@@ -2,5 +2,5 @@
 <robot xmlns:xacro="http://www.ros.org/wiki/xacro" name="lidar">
   <!-- Ссылка -->
-  <link name="lidar">
+  <link name="laser_frame">
     <visual>
       <geometry>
@@ -21,5 +21,5 @@
   <joint name="base_lidar_joint" type="fixed">
     <parent link="base_link"/>
-    <child link="lidar"/>
+    <child link="laser_frame"/>
     <origin xyz="0 0 ${lidar_offset_z}" rpy="0 0 0"/>
   </joint>
